Commit message: Small engine tests with trajectory optimization tests

File: splatsim/robot_definitions/urdf/sisbot.urdf (robot description, URDF)
Before this commit: robot sisbot, 21 links, 20 joints
Links:
- removed link dummy_center_indicator_link
Joints:
- removed joint dummy_center_fixed_joint

Commit message: Add wrist cam to ur5 robot (sisbot)

File: splatsim/robot_definitions/urdf/sisbot.urdf (robot description, URDF)
Before this commit: robot sisbot, 20 links, 19 joints
Links:
- added link wrist_camera_link
- added link wrist_camera_vis_x_link; visual cylinder length=0.1 radius=0.005
- added link wrist_camera_vis_y_link; visual cylinder length=0.1 radius=0.005
- added link wrist_camera_vis_z_link; visual cylinder length=0.1 radius=0.005
Joints:
- added joint wrist_camera_vis_joint: type fixed, parent robotiq_arg2f_base_link, child wrist_camera_link, origin xyz=-0.1 0 0.05 rpy=0 0 -1.57
- added joint wrist_camera_vis_x_joint: type fixed, parent wrist_camera_link, child wrist_camera_vis_x_link, origin xyz=0 0 0 rpy=0 0 0
- added joint wrist_camera_vis_y_joint: type fixed, parent wrist_camera_link, child wrist_camera_vis_y_link, origin xyz=0 0 0 rpy=0 0 0
- added joint wrist_camera_vis_z_joint: type fixed, parent wrist_camera_link, child wrist_camera_vis_z_link, origin xyz=0 0 0 rpy=0 0 0

Commit message: move ur5 wrist camera back; WIP camera datastructure changing

File: splatsim/robot_definitions/urdf/sisbot.urdf (robot description, URDF)
Before this commit: robot sisbot, 24 links, 23 joints
Joints:
- joint wrist_camera_vis_joint: origin xyz=-0.1 0 0.05 rpy=0 0 -1.57 -> xyz=-0.1 0 -0.05 rpy=0 0 -1.57

Commit message: Move gopro wrist cam on sisbot downwards to match real robot

File: splatsim/robot_definitions/urdf/sisbot.urdf (robot description, URDF)
Before this commit: robot sisbot, 24 links, 23 joints
Joints:
- joint wrist_camera_vis_joint: origin xyz=-0.1 0 -0.05 rpy=0 0 -1.57 -> xyz=-0.1 0 -0.05 rpy=-0.3141 0 -1.57

Commit message: Fix wrist cam phasing through box surfaces; Support global_scaling for splat rendering

File: splatsim/robot_definitions/urdf/sisbot.urdf (robot description, URDF)
Before this commit: robot sisbot, 24 links, 23 joints
Links:
- link wrist_camera_link: geometry collision box size=0.072 0.051 0.034; visual box size=0.072 0.051 0.034
Joints:
- joint wrist_camera_vis_joint: origin xyz=-0.1 0 -0.05 rpy=-0.3141 0 -1.57 -> xyz=-0.1 0 -0.0 rpy=-0.3141 0 -1.57
