Commit message: Misc: keyboard agent, URDF, rendering, calibration
Updates keyboard_interface_agent + run_env_sim launcher behavior, sisbot
URDF collision-shape tweaks, gsplat_renderer adjustments, and a saved
calibration output from calibrate_camera_intrinsics.

Co-Authored-By: Claude Opus 4.7 <noreply@anthropic.com>

File: splatsim/robot_definitions/urdf/sisbot.urdf (robot description, URDF)
Before this commit: robot sisbot, 24 links, 23 joints
Joints:
- joint wrist_camera_vis_joint: origin xyz=-0.1 0 -0.0 rpy=-0.3141 0 -1.57 -> xyz=-0.1 0 -0.0 rpy=0 0 -1.57

Commit message: Fix gripper mimic actuation and reset/teleport reliability
Gripper: stop position-holding the Robotiq mimic child joints (teleport_
joint_state / command_joint_state hold arm DOFs only) and disable their
physics self-collision in setup_gripper so the JOINT_GEAR mimic can open/
close; uncomment the gripper-base collision STL for RRT. Capture the splat
transform reference (initial_link_poses) at initial_joint_positions BEFORE
the settle loop so the open URDF renders an open splat. run_env_sim no
longer strips the gripper element from the action. Slider agent defaults
open with a 0..1 gripper control.

Reset: randomize_ee_pose returns None (and callers re-randomize) instead of
committing a colliding pose, ending the post-reset stutter with stale-closed
gripper; small_engine opens the gripper on every reset.

Also add DEFAULT_ROBOT_NAME, wrist_cam_ver=2 default, in_collision
clearance plumbing, and the audited SELF_COLLISION_SKIP_PAIRS.

Co-Authored-By: Claude Opus 4.8 <noreply@anthropic.com>

File: splatsim/robot_definitions/urdf/sisbot.urdf (robot description, URDF)
Before this commit: robot sisbot, 24 links, 23 joints
Links:
- link robotiq_arg2f_base_link: geometry collision mesh filename=collision/robotiq_arg2f_base_link.stl; visual mesh filename=visual/robotiq_arg2f_85_base_link.dae scale=0.001 0.001 0.001
Joints:
- joint wrist_camera_vis_joint: origin xyz=-0.1 0 -0.0 rpy=0 0 -1.57 -> xyz=-0.1 -0.0 -0.035 rpy=-0.3141 0 -1.57
