Commit message: floating gripper: vine-splat variant, TCP frame fix, PyBullet compositing
Adds VineFloatingGripperPybulletRobotServer — the floating-gripper replay
rendered inside the scanned grape-vine splat, with the (unscanned) gripper
composited in from PyBullet against the splat's expected depth.

- gsplat_renderer: opt-in RGB+ED so callers can get expected depth for the
  composite; off by default since almost every render only wants colour.
- base server: COMPOSITE_PYBULLET_ROBOT / COMPOSITE_DEPTH_SLACK_M, the
  depth-composite path, and read-only lerobot dataset init.
- floating_gripper.urdf: correct the TCP mount — the UMI tcp_pose frame has
  -Y = approach and +X = finger-opening (verified against the 2026-08-20
  ground video), not +Z = approach.
- rrt retiming: handoff plans (start_vel given) take the jerk-limited onset
  at any handoff speed, including ~0; stalled takeovers were launching at
  cruise within one tick and producing unfollowable labels.
- gui: wait_until_ready so pre-build setter writes stop silently vanishing;
  seed the eval-benchmark repo-id field from the server flag.
- launch_nodes: wire the new variant; sync_physics_to_client now defaults on
  so rollout dynamics stop depending on GPU load.

Co-Authored-By: Claude Opus 5 (1M context) <noreply@anthropic.com>

File: splatsim/robot_definitions/urdf/floating_gripper.urdf (robot description, URDF)
Before this commit: robot floating_gripper, 20 links, 19 joints
Joints:
- joint arm_gripper_joint: origin xyz=0.0 0.0 -0.15 rpy=0.0 0.0 0.0 -> xyz=0.0 0.15 0.0 rpy=1.5707963267948966 1.5707963267948966 0.0
