Commit message: placement: gripper sliders, named scenarios; Play on by default; panda wrist camera beside the hand
- Robot Placement panel: one slider per gripper command (0 open .. 1
  closed) for every arm; a scenario name field with Save / Load scenario
  (data/scenarios/<env>__<robot>__<name>.json, loading pins it for resets
  and syncs the sliders from the robot's actual state), plus "Save as robot
  default (yaml)" for what Save placement used to do. Scenario files now
  carry the robot's base pose.
- launch_nodes: --scenario <name> (default "default"); the old unnamed
  cache file is renamed to __default on first launch.
- Play starts on and follows the mode: off entering trajectory
  generation, on entering anything else. Eval-benchmark playback is
  unaffected (periodic rendering never fires in event-rendered modes).
- panda.urdf: wrist_camera_link on the side of the hand (+x, tilted 15 deg
  toward the fingers) with RGB axis cylinders like the UR5's; the camera
  no longer stares at the closed fingers. dual_panda regenerated from it.

Co-Authored-By: Claude Fable 5.1 <noreply@anthropic.com>

File: data/assets/dual_panda/dual_panda.urdf (robot description, URDF)
Before this commit: robot dual_panda, 27 links, 26 joints
Links:
- added link left_wrist_camera_link; collision box size=0.02 0.03 0.02; visual box size=0.02 0.03 0.02
- added link left_wrist_camera_vis_x_link; visual cylinder length=0.1 radius=0.004
- added link left_wrist_camera_vis_y_link; visual cylinder length=0.1 radius=0.004
- added link left_wrist_camera_vis_z_link; visual cylinder length=0.1 radius=0.004
- added link right_wrist_camera_link; collision box size=0.02 0.03 0.02; visual box size=0.02 0.03 0.02
- added link right_wrist_camera_vis_x_link; visual cylinder length=0.1 radius=0.004
- added link right_wrist_camera_vis_y_link; visual cylinder length=0.1 radius=0.004
- added link right_wrist_camera_vis_z_link; visual cylinder length=0.1 radius=0.004
Joints:
- added joint left_wrist_camera_joint: type fixed, parent left_panda_hand, child left_wrist_camera_link, origin xyz=0.06 0 0.02 rpy=0 -0.2618 0
- added joint left_wrist_camera_vis_x_joint: type fixed, parent left_wrist_camera_link, child left_wrist_camera_vis_x_link, origin xyz=0 0 0 rpy=0 0 0
- added joint left_wrist_camera_vis_y_joint: type fixed, parent left_wrist_camera_link, child left_wrist_camera_vis_y_link, origin xyz=0 0 0 rpy=0 0 0
- added joint left_wrist_camera_vis_z_joint: type fixed, parent left_wrist_camera_link, child left_wrist_camera_vis_z_link, origin xyz=0 0 0 rpy=0 0 0
- added joint right_wrist_camera_joint: type fixed, parent right_panda_hand, child right_wrist_camera_link, origin xyz=0.06 0 0.02 rpy=0 -0.2618 0
- added joint right_wrist_camera_vis_x_joint: type fixed, parent right_wrist_camera_link, child right_wrist_camera_vis_x_link, origin xyz=0 0 0 rpy=0 0 0
- added joint right_wrist_camera_vis_y_joint: type fixed, parent right_wrist_camera_link, child right_wrist_camera_vis_y_link, origin xyz=0 0 0 rpy=0 0 0
- added joint right_wrist_camera_vis_z_joint: type fixed, parent right_wrist_camera_link, child right_wrist_camera_vis_z_link, origin xyz=0 0 0 rpy=0 0 0

File: data/assets/panda/panda.urdf (robot description, URDF)
Before this commit: robot panda, 13 links, 12 joints
Links:
- added link wrist_camera_link; collision box size=0.02 0.03 0.02; visual box size=0.02 0.03 0.02
- added link wrist_camera_vis_x_link; visual cylinder length=0.1 radius=0.004
- added link wrist_camera_vis_y_link; visual cylinder length=0.1 radius=0.004
- added link wrist_camera_vis_z_link; visual cylinder length=0.1 radius=0.004
Joints:
- added joint wrist_camera_joint: type fixed, parent panda_hand, child wrist_camera_link, origin xyz=0.06 0 0.02 rpy=0 -0.2618 0
- added joint wrist_camera_vis_x_joint: type fixed, parent wrist_camera_link, child wrist_camera_vis_x_link, origin xyz=0 0 0 rpy=0 0 0
- added joint wrist_camera_vis_y_joint: type fixed, parent wrist_camera_link, child wrist_camera_vis_y_link, origin xyz=0 0 0 rpy=0 0 0
- added joint wrist_camera_vis_z_joint: type fixed, parent wrist_camera_link, child wrist_camera_vis_z_link, origin xyz=0 0 0 rpy=0 0 0

Commit message: panda: elbow camera as a URDF link with RGB axes, like the wrist camera
Co-Authored-By: Claude Fable 5.1 <noreply@anthropic.com>

File: data/assets/dual_panda/dual_panda.urdf (robot description, URDF)
Before this commit: robot dual_panda, 35 links, 34 joints
Links:
- added link left_elbow_camera_link; visual box size=0.02 0.03 0.02
- added link left_elbow_camera_vis_x_link; visual cylinder length=0.1 radius=0.004
- added link left_elbow_camera_vis_y_link; visual cylinder length=0.1 radius=0.004
- added link left_elbow_camera_vis_z_link; visual cylinder length=0.1 radius=0.004
- added link right_elbow_camera_link; visual box size=0.02 0.03 0.02
- added link right_elbow_camera_vis_x_link; visual cylinder length=0.1 radius=0.004
- added link right_elbow_camera_vis_y_link; visual cylinder length=0.1 radius=0.004
- added link right_elbow_camera_vis_z_link; visual cylinder length=0.1 radius=0.004
Joints:
- added joint left_elbow_camera_joint: type fixed, parent left_panda_link4, child left_elbow_camera_link, origin xyz=0 0 0.1 rpy=1.5708 0 0
- added joint left_elbow_camera_vis_x_joint: type fixed, parent left_elbow_camera_link, child left_elbow_camera_vis_x_link, origin xyz=0 0 0 rpy=0 0 0
- added joint left_elbow_camera_vis_y_joint: type fixed, parent left_elbow_camera_link, child left_elbow_camera_vis_y_link, origin xyz=0 0 0 rpy=0 0 0
- added joint left_elbow_camera_vis_z_joint: type fixed, parent left_elbow_camera_link, child left_elbow_camera_vis_z_link, origin xyz=0 0 0 rpy=0 0 0
- added joint right_elbow_camera_joint: type fixed, parent right_panda_link4, child right_elbow_camera_link, origin xyz=0 0 0.1 rpy=1.5708 0 0
- added joint right_elbow_camera_vis_x_joint: type fixed, parent right_elbow_camera_link, child right_elbow_camera_vis_x_link, origin xyz=0 0 0 rpy=0 0 0
- added joint right_elbow_camera_vis_y_joint: type fixed, parent right_elbow_camera_link, child right_elbow_camera_vis_y_link, origin xyz=0 0 0 rpy=0 0 0
- added joint right_elbow_camera_vis_z_joint: type fixed, parent right_elbow_camera_link, child right_elbow_camera_vis_z_link, origin xyz=0 0 0 rpy=0 0 0

File: data/assets/panda/panda.urdf (robot description, URDF)
Before this commit: robot panda, 17 links, 16 joints
Links:
- added link elbow_camera_link; visual box size=0.02 0.03 0.02
- added link elbow_camera_vis_x_link; visual cylinder length=0.1 radius=0.004
- added link elbow_camera_vis_y_link; visual cylinder length=0.1 radius=0.004
- added link elbow_camera_vis_z_link; visual cylinder length=0.1 radius=0.004
Joints:
- added joint elbow_camera_joint: type fixed, parent panda_link4, child elbow_camera_link, origin xyz=0 0 0.1 rpy=1.5708 0 0
- added joint elbow_camera_vis_x_joint: type fixed, parent elbow_camera_link, child elbow_camera_vis_x_link, origin xyz=0 0 0 rpy=0 0 0
- added joint elbow_camera_vis_y_joint: type fixed, parent elbow_camera_link, child elbow_camera_vis_y_link, origin xyz=0 0 0 rpy=0 0 0
- added joint elbow_camera_vis_z_joint: type fixed, parent elbow_camera_link, child elbow_camera_vis_z_link, origin xyz=0 0 0 rpy=0 0 0
